Commit message: Add files via upload

File: barrett_hand_target.urdf (robot description, URDF)
Before this commit: robot BarrettHand-280, 16 links, 15 joints
Links:
- link contact_point_base: geometry collision mesh filename=/urdf_model/small_cube.obj scale=1 1 1; visual mesh filename=/urdf_model/contact point.obj scale=1 1 1
- link contact_point_f1_dist: geometry collision mesh filename=/urdf_model/contact point.obj scale=1 1 1; visual mesh filename=/urdf_model/contact point.obj scale=1 1 1
- link contact_point_f1_med: geometry collision mesh filename=/urdf_model/contact point.obj scale=1 1 1; visual mesh filename=/urdf_model/contact point.obj scale=1 1 1
- link contact_point_f2_dist: geometry collision mesh filename=/urdf_model/contact point.obj scale=1 1 1; visual mesh filename=/urdf_model/contact point.obj scale=1 1 1
- link contact_point_f2_med: geometry collision mesh filename=/urdf_model/contact point.obj scale=1 1 1; visual mesh filename=/urdf_model/contact point.obj scale=1 1 1
- link contact_point_f3_dist: geometry collision mesh filename=/urdf_model/contact point.obj scale=1 1 1; visual mesh filename=/urdf_model/contact point.obj scale=1 1 1
- link contact_point_f3_med: geometry collision mesh filename=/urdf_model/contact point.obj scale=1 1 1; visual mesh filename=/urdf_model/contact point.obj scale=1 1 1
